Commit message: last change

File: lucy/description/lucy.body.xacro (robot description, xacro)
@@ -74,10 +74,10 @@
         </visual>
     </link>
-    <joint name="base_lidar_joint" type="revolute">
+    <joint name="base_lidar_joint" type="fixed">
         <parent link="base_link" />
         <child link="lidar_box_link" />
         <origin xyz="0 0 0.22" rpy="0 0 0" />
-        <axis xyz="0 1 0" />
-        <limit lower="-0.523" upper="0.523" effort="10" velocity="1" />
+        <!-- <axis xyz="0 1 0" /> -->
+        <!-- <limit lower="-0.523" upper="0.523" effort="10" velocity="1" /> -->
     </joint>
     <link name="lidar_box_link">

File: lucy/description/lucy.control.xacro (robot description, xacro)
@@ -6,9 +6,9 @@
       <param name="left_wheel_name">left_wheel_joint</param>
       <param name="right_wheel_name">right_wheel_joint</param>
-      <param name="loop_rate">50</param>
+      <param name="loop_rate">8</param>
       <param name="device">/dev/ttyACM0</param>
       <param name="baud_rate">115200</param>
       <param name="timeout">1000</param>
-      <param name="enc_counts_per_rev">546</param>
+      <param name="enc_counts_per_rev">435</param>
     </hardware>
     <joint name="left_wheel_joint">
